File: kicad/bcm-mixer.kicad_pcb (KiCad board)
At the start: 2 copper layers, 142 x 108.5 mm, 99 parts, among them J1 AudioJack2_SwitchT, J10 Conn_01x08_Pin, J11 Conn_01x08_Socket, J12 Conn_01x08_Socket, J13 Conn_01x08_Pin, J14 Conn_01x06_Pin, J15 Conn_01x06_Socket, J16 Conn_01x06_Socket, J17 Conn_01x06_Pin, J2 AudioJack2_SwitchT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

Commit message: Updating everything and adding gerbers
Parts:
- added H1: MountingHole_Pad, Rumblesan_Standard_Parts:MountingHole_3.2mm_M3_DIN965_Pad, F.Cu at (68.5, 57.2)
- added H2: MountingHole_Pad, Rumblesan_Standard_Parts:MountingHole_3.2mm_M3_DIN965_Pad, F.Cu at (140.5, 57.2)
- added H3: MountingHole_Pad, Rumblesan_Standard_Parts:MountingHole_3.2mm_M3_DIN965_Pad, F.Cu at (85.5, 143.0)
- added H4: MountingHole_Pad, Rumblesan_Standard_Parts:MountingHole_3.2mm_M3_DIN965_Pad, F.Cu at (157.5, 143.0)
- C1, C13, C17, C19, C20, C21, C26, C7: footprint Capacitor_THT:CP_Radial_D5.0mm_P2.00mm -> Rumblesan_Standard_Parts:CP_Radial_D5.0mm_P2.00mm
- moved R36 10.2 mm to (135.6, 124.2), turned to -90 degrees
- moved R41 10.2 mm to (106.9, 124.5), turned to -90 degrees
- moved R5 10.2 mm to (110.0, 134.6), turned to 90 degrees
- moved R1 10.2 mm to (170.7, 56.9), turned to -90 degrees
- moved R10 10.2 mm to (161.5, 123.2), turned to 90 degrees
- moved R11 10.2 mm to (167.6, 123.2), turned to 90 degrees
- moved R12 10.2 mm to (158.5, 113.0), turned to -90 degrees
- moved R13 10.2 mm to (164.6, 113.0), turned to -90 degrees
- moved R14 10.2 mm to (117.0, 136.1), turned to -90 degrees
- moved R15 10.2 mm to (116.8, 122.4), turned to 90 degrees
- moved R16 10.2 mm to (145.0, 123.3), turned to 90 degrees
- moved R17 10.2 mm to (151.1, 123.3), turned to 90 degrees
- moved R18 10.2 mm to (129.0, 69.3), turned to -90 degrees
- moved R19 10.2 mm to (135.1, 69.3), turned to -90 degrees
- moved R2 10.2 mm to (127.5, 146.3), turned to 90 degrees
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Connections:
- R1 pad 1: /CHAN1_INPUT_MAIN -> GND
- R1 pad 2: GND -> /CHAN1_INPUT_MAIN
- R10 pad 1: /CHAN1_PAN_CW_MAIN -> /Mono Channel 1/OUTPUT
- R10 pad 2: /Mono Channel 1/OUTPUT -> /CHAN1_PAN_CW_MAIN
- R11 pad 1: /CHAN1_PAN_CCW_MAIN -> /Mono Channel 1/OUTPUT
- R11 pad 2: /Mono Channel 1/OUTPUT -> /CHAN1_PAN_CCW_MAIN
- R12 pad 1: MAIN_BUS_L -> /CHAN1_PAN_CW_MAIN
- R12 pad 2: /CHAN1_PAN_CW_MAIN -> MAIN_BUS_L
- R13 pad 1: MAIN_BUS_R -> /CHAN1_PAN_CCW_MAIN
- R13 pad 2: /CHAN1_PAN_CCW_MAIN -> MAIN_BUS_R
- R14 pad 1: /Main Channel/L_OUT -> Net-(U3C--)
- R14 pad 2: Net-(U3C--) -> /Main Channel/L_OUT
- R15 pad 1: /Main Channel/R_OUT -> Net-(U3B--)
- R15 pad 2: Net-(U3B--) -> /Main Channel/R_OUT
- R16 pad 1: /CHAN2_PAN_CW_MAIN -> /Mono Channel 2/OUTPUT
- R16 pad 2: /Mono Channel 2/OUTPUT -> /CHAN2_PAN_CW_MAIN
- R17 pad 1: /CHAN2_PAN_CCW_MAIN -> /Mono Channel 2/OUTPUT
- R17 pad 2: /Mono Channel 2/OUTPUT -> /CHAN2_PAN_CCW_MAIN
- R18 pad 1: Net-(U2A--) -> Net-(C13-Pad2)
- R18 pad 2: Net-(C13-Pad2) -> Net-(U2A--)
- R19 pad 1: /CHAN3_L_OUTPUT_MAIN -> Net-(U2A--)
- R19 pad 2: Net-(U2A--) -> /CHAN3_L_OUTPUT_MAIN
- R2 pad 1: /MAIN_L_LEVEL_CW_MAIN -> MAIN_BUS_L
- R2 pad 2: MAIN_BUS_L -> /MAIN_L_LEVEL_CW_MAIN
- R20 pad 1: /CHAN3_L_INPUT_MAIN -> GND
- R20 pad 2: GND -> /CHAN3_L_INPUT_MAIN
- R21 pad 1: /CHAN3_R_INPUT_MAIN -> GND
- R21 pad 2: GND -> /CHAN3_R_INPUT_MAIN
- R22 pad 1: Net-(U2B--) -> Net-(C17-Pad2)
- R22 pad 2: Net-(C17-Pad2) -> Net-(U2B--)
- R23 pad 1: /CHAN3_R_OUTPUT_MAIN -> Net-(U2B--)
- R23 pad 2: Net-(U2B--) -> /CHAN3_R_OUTPUT_MAIN
- R24 pad 1: MAIN_BUS_R -> /CHAN2_PAN_CCW_MAIN
- R24 pad 2: /CHAN2_PAN_CCW_MAIN -> MAIN_BUS_R
- R25 pad 1: MAIN_BUS_L -> /CHAN2_PAN_CW_MAIN
- R25 pad 2: /CHAN2_PAN_CW_MAIN -> MAIN_BUS_L
- R26 pad 1: /CHAN2_INPUT_MAIN -> GND
- R26 pad 2: GND -> /CHAN2_INPUT_MAIN
- R27 pad 1: /CHAN2_GAIN_CENTER_MAIN -> Net-(C21-Pad1)
- R27 pad 2: Net-(C21-Pad1) -> /CHAN2_GAIN_CENTER_MAIN
- R28 pad 1: /CHAN2_LEVEL_CW_MAIN -> /CHAN2_GAIN_CCW_MAIN
- R28 pad 2: /CHAN2_GAIN_CCW_MAIN -> /CHAN2_LEVEL_CW_MAIN
- R29 pad 1: Net-(U4B--) -> /CHAN2_LEVEL_CENTER_MAIN
- R29 pad 2: /CHAN2_LEVEL_CENTER_MAIN -> Net-(U4B--)
- R3 pad 1: /MAIN_R_LEVEL_CW_MAIN -> MAIN_BUS_R
- R3 pad 2: MAIN_BUS_R -> /MAIN_R_LEVEL_CW_MAIN
- R30 pad 1: Net-(C25-Pad2) -> Net-(U4B--)
- R30 pad 2: Net-(U4B--) -> Net-(C25-Pad2)
- R31 pad 1: MAIN_BUS_L -> Net-(J14-Pin_5)
- R31 pad 2: Net-(J14-Pin_5) -> MAIN_BUS_L
- R32 pad 1: MAIN_BUS_R -> Net-(J14-Pin_3)
- R32 pad 2: Net-(J14-Pin_3) -> MAIN_BUS_R
- R35 pad 1: MAIN_BUS_L -> Net-(J8-Pin_3)
- R35 pad 2: Net-(J8-Pin_3) -> MAIN_BUS_L
- R36 pad 1: Net-(J8-Pin_7) -> MAIN_BUS_R
- R36 pad 2: MAIN_BUS_R -> Net-(J8-Pin_7)
- R4 pad 1: Net-(U3C--) -> /MAIN_L_LEVEL_CENTER_MAIN
- R4 pad 2: /MAIN_L_LEVEL_CENTER_MAIN -> Net-(U3C--)
- R40 pad 1: /L_OUT_MAIN -> /Main Channel/L_OUT
- R40 pad 2: /Main Channel/L_OUT -> /L_OUT_MAIN
- R41 pad 1: /R_OUT_MAIN -> /Main Channel/R_OUT
- R41 pad 2: /Main Channel/R_OUT -> /R_OUT_MAIN
- R5 pad 1: Net-(U3B--) -> /MAIN_R_LEVEL_CENTER_MAIN
- R5 pad 2: /MAIN_R_LEVEL_CENTER_MAIN -> Net-(U3B--)
- R6 pad 1: /CHAN1_GAIN_CENTER_MAIN -> Net-(C1-Pad1)
- R6 pad 2: Net-(C1-Pad1) -> /CHAN1_GAIN_CENTER_MAIN
- R7 pad 1: /CHAN1_LEVEL_CW_MAIN -> /CHAN1_GAIN_CCW_MAIN
- R7 pad 2: /CHAN1_GAIN_CCW_MAIN -> /CHAN1_LEVEL_CW_MAIN
- R8 pad 1: Net-(U1B--) -> /CHAN1_LEVEL_CENTER_MAIN
- R8 pad 2: /CHAN1_LEVEL_CENTER_MAIN -> Net-(U1B--)
- R9 pad 1: Net-(C6-Pad2) -> Net-(U1B--)
- R9 pad 2: Net-(U1B--) -> Net-(C6-Pad2)
- RV3 pad 4: (no net) -> unconnected-(RV3-Pad4)
- RV3 pad 5: (no net) -> unconnected-(RV3-Pad5)
- RV3 pad 6: (no net) -> GND
- RV6 pad 4: (no net) -> unconnected-(RV6-Pad4)
- RV6 pad 5: (no net) -> unconnected-(RV6-Pad5)
- RV6 pad 6: (no net) -> GND
Routing:
- net VCC: track 154.6 -> 153.1 mm
- net VEE: track 202.5 -> 203.7 mm
- net Net-(D1-A): track 10.8 -> 11.6 mm
