File: kicad/bcm-mixer-panel.kicad_pcb (KiCad board)
At the start: 2 copper layers, 70.8 x 128.5 mm, 5 parts

Commit message: Updating for revision 2
Parts:
- added H5: MountingHole, MountingHole:MountingHole_3.2mm_M3_DIN965, F.Cu at (83.5, 143.0)
Other:
- outline, holes or cut-outs redrawn
