File: kicad/mono-channel.kicad_sch (KiCad schematic)
At the start: 12 parts, among them U1 TL072

Commit message: Updating everything and adding gerbers
Parts:
- C1, C7: footprint Capacitor_THT:CP_Radial_D5.0mm_P2.00mm -> Rumblesan_Standard_Parts:CP_Radial_D5.0mm_P2.00mm; symbol Standard_Parts:C_Polarized -> Rumblesan_Standard_Parts:C_Polarized
- C5, C6, C8, C9: symbol Standard_Parts:C -> Rumblesan_Standard_Parts:C
- R1, R6, R7, R8, R9: symbol Standard_Parts:R -> Rumblesan_Standard_Parts:R
Connections:
- net GAIN_POT_CCW: now also R7.1; no longer R7.2
- net GAIN_POT_CENTER: now also R6.2; no longer R6.1
- net GND: now also R1.1; no longer R1.2
- net INPUT: now also R1.2; no longer R1.1
- net LEVEL_POT_CENTER: now also R8.1; no longer R8.2
- net LEVEL_POT_CW: now also R7.2; no longer R7.1
- net at C6.2, C7.2, U1.7: now also R9.2; no longer R9.1
- net at C6.1, U1.6 (-): now also R8.2, R9.1; no longer R8.1, R9.2
- net at C1.1: now also R6.1; no longer R6.2
Changed lines of the file:
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@@
 	)
 	(symbol
-		(lib_id "Standard_Parts:C")
+		(lib_id "Rumblesan_Standard_Parts:C")
 		(at 92.71 68.58 90)
 		(unit 1)
@@
 	)
 	(symbol
-		(lib_id "Standard_Parts:C_Polarized")
+		(lib_id "Rumblesan_Standard_Parts:C_Polarized")
 		(at 184.15 88.9 270)
 		(unit 1)
@@
 			)
 		)
-		(property "Footprint" "Capacitor_THT:CP_Radial_D5.0mm_P2.00mm"
+		(property "Footprint" "Rumblesan_Standard_Parts:CP_Radial_D5.0mm_P2.00mm"
 			(at 184.15 95.25 90)
 			(effects
@@
 	)
 	(symbol
-		(lib_id "Standard_Parts:C")
+		(lib_id "Rumblesan_Standard_Parts:C")
 		(at 161.29 63.5 90)
 		(unit 1)
@@
 	)
 	(symbol
-		(lib_id "Standard_Parts:C")
+		(lib_id "Rumblesan_Standard_Parts:C")
 		(at 92.71 125.73 180)
 		(unit 1)
@@
 	)
 	(symbol
-		(lib_id "Standard_Parts:R")
+		(lib_id "Rumblesan_Standard_Parts:R")
 		(at 140.97 86.36 90)
 		(unit 1)
@@
 	)
 	(symbol
-		(lib_id "Standard_Parts:C_Polarized")
+		(lib_id "Rumblesan_Standard_Parts:C_Polarized")
 		(at 58.42 77.47 270)
 		(unit 1)
@@
 			)
 		)
-		(property "Footprint" "Capacitor_THT:CP_Radial_D5.0mm_P2.00mm"
+		(property "Footprint" "Rumblesan_Standard_Parts:CP_Radial_D5.0mm_P2.00mm"
 			(at 58.42 83.82 90)
 			(effects
@@
 	)
 	(symbol
-		(lib_id "Standard_Parts:R")
+		(lib_id "Rumblesan_Standard_Parts:R")
 		(at 69.85 77.47 90)
 		(unit 1)
@@
 	)
 	(symbol
-		(lib_id "Standard_Parts:R")
+		(lib_id "Rumblesan_Standard_Parts:R")
 		(at 161.29 76.2 90)
 		(unit 1)
@@
 	)
 	(symbol
-		(lib_id "Standard_Parts:C")
+		(lib_id "Rumblesan_Standard_Parts:C")
 		(at 92.71 135.89 180)
 		(unit 1)
@@
 	)
 	(symbol
-		(lib_id "Standard_Parts:R")
+		(lib_id "Rumblesan_Standard_Parts:R")
 		(at 93.98 57.15 90)
 		(unit 1)
@@
 	)
 	(symbol
-		(lib_id "Standard_Parts:R")
+		(lib_id "Rumblesan_Standard_Parts:R")
 		(at 50.8 85.09 180)
 		(unit 1)

Commit message: Updating for revision 2
Parts:
- C1: value 1uF -> 10uF
- R6: value 2k2 -> 10k
- R8, R9: value 10k -> 100k
Connections:
- net INPUT: now also C1.1; no longer C1.2
- net at R6.1: now also C1.2; no longer C1.1
Other:
- note added: "100k gain pot with 10k resistors means 11 times gain equals 20.8 db"
- note added: "lowpass filter freq 723kHz at min gain 65kHz at max gain"
- note added: "lowpass filter freq 72kHz"
- moved on the sheet: C1
Changed lines of the file:
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@@
+		)
+	)
+	(text "100k gain pot with 10k resistors\nmeans 11 times gain\nequals 20.8 db"
+		(exclude_from_sim no)
+		(at 107.188 45.72 0)
+		(effects
+			(font
+				(size 1.27 1.27)
+			)
+		)
+	)
+	(text "lowpass filter freq 72kHz"
+		(exclude_from_sim no)
+		(at 189.484 69.342 0)
+		(effects
+			(font
+				(size 1.27 1.27)
+			)
+		)
+	)
+	(text "lowpass filter freq\n723kHz at min gain\n65kHz at max gain"
+		(exclude_from_sim no)
+		(at 118.364 62.484 0)
+		(effects
+			(font
+				(size 1.27 1.27)
+			)
 		)
 	)
@@
 			)
 		)
-		(property "Value" "10k"
+		(property "Value" "100k"
 			(at 140.97 82.55 90)
 			(effects
@@
 	(symbol
 		(lib_id "Rumblesan_Standard_Parts:C_Polarized")
-		(at 58.42 77.47 270)
-		(unit 1)
-		(exclude_from_sim no)
-		(in_bom yes)
-		(on_board yes)
-		(dnp no)
-		(fields_autoplaced yes)
+		(at 58.42 77.47 90)
+		(mirror x)
+		(unit 1)
+		(exclude_from_sim no)
+		(in_bom yes)
+		(on_board yes)
+		(dnp no)
 		(property "Reference" "C1"
-			(at 59.309 69.85 90)
-			(effects
-				(font
-					(size 1.27 1.27)
-				)
-			)
-		)
-		(property "Value" "1uF"
-			(at 59.309 72.39 90)
+			(at 57.531 69.85 90)
+			(effects
+				(font
+					(size 1.27 1.27)
+				)
+			)
+		)
+		(property "Value" "10uF"
+			(at 57.531 72.39 90)
 			(effects
 				(font
@@
 		)
 		(property "Spec" "electrolytic"
+			(at 62.23 81.28 90)
+			(effects
+				(font
+					(size 1.27 1.27)
+				)
+				(hide yes)
+			)
+		)
+		(property "Tolerance" "20%"
+			(at 50.8 81.28 90)
+			(effects
+				(font
+					(size 1.27 1.27)
+				)
+				(hide yes)
+			)
+		)
+		(property "Voltage" "50v"
 			(at 54.61 81.28 90)
-			(effects
-				(font
-					(size 1.27 1.27)
-				)
-				(hide yes)
-			)
-		)
-		(property "Tolerance" "20%"
-			(at 66.04 81.28 90)
-			(effects
-				(font
-					(size 1.27 1.27)
-				)
-				(hide yes)
-			)
-		)
-		(property "Voltage" "50v"
-			(at 62.23 81.28 90)
 			(effects
 				(font
@@
 			)
 		)
-		(property "Value" "2k2"
+		(property "Value" "10k"
 			(at 69.85 73.66 90)
 			(effects
@@
 			)
 		)
-		(property "Value" "10k"
+		(property "Value" "100k"
 			(at 161.29 72.39 90)
 			(effects
